File: Storage.kicad_sch (KiCad schematic)
At the start: 4 parts, among them SW1 SW_Push, U3 W25Q128JVS

Commit message: Restore
Parts:
- R6, R7: footprint (none) -> Resistor_SMD:R_0402_1005Metric
- SW1: footprint (none) -> JonasLib-Git:smd_switch_sunrom4388
Changed lines of the file:
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@@
 			)
 		)
-		(property "Footprint" ""
+		(property "Footprint" "Resistor_SMD:R_0402_1005Metric"
 			(at 234.442 33.02 90)
 			(effects
@@
 			)
 		)
-		(property "Footprint" ""
+		(property "Footprint" "Resistor_SMD:R_0402_1005Metric"
 			(at 228.6 39.878 90)
 			(effects
@@
 			)
 		)
-		(property "Footprint" ""
+		(property "Footprint" "JonasLib-Git:smd_switch_sunrom4388"
 			(at 218.44 33.02 0)
 			(effects
