File: power.kicad_sch (KiCad schematic)
At the start: 18 parts, among them J1 USB_C_Receptacle_USB2.0_14P, U2 NCP1117-3.3_SOT223

Commit message: Restore
Parts:
- added C20: 100nF, Capacitor_SMD:C_0402_1005Metric, symbol Device:C
- C1, C10, C11, C12, C13, C14, C2, C3, C4, C5, C6, C7, C8, C9: footprint (none) -> Capacitor_SMD:C_0402_1005Metric
- J1: footprint (none) -> Connector_USB:USB_C_Receptacle_HRO_TYPE-C-31-M-12
- R1, R2: footprint (none) -> Resistor_SMD:R_0402_1005Metric
Connections:
- net +3V3: now also C20.1
- net GND: now also C20.2
Other:
- moved on the sheet: C1, C2, C3, C4, C5, C6, C7, C8, C9
